File: optical_pcb_v2.kicad_sch (KiCad schematic)
At the start: 14 parts

Commit message: updated to v2
Connections:
- net GND: now reaches SMP1.2
- net GND: now also SMP1.3, SMP1.4, SMP1.5, SMP2.2, SMP2.3, SMP2.4, SMP2.5, SMP3.2, SMP3.3, SMP3.4, SMP3.5, SMP4.2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
